File: antartix-arty-controller.sch (KiCad schematic (older format))
At the start: 13 parts

Commit message: Add power switches, add current monitor circuits
Parts:
- added C?: C_100n_0402, antmicro-footprints:0402-cap, symbol antmicroCapacitors0402:C_100n_0402
- added R? (x3): R_0R01_1206, antmicro-footprints:1206-res, symbol antmicroResistorsmisc:R_0R01_1206
- added U? (x3): TPS2051BDBVR, antmicro-footprints:SOT-753, symbol antmicroPMICPowerDistributionSwitchesLoadDrivers:TPS2051BDBVR
Connections:
- net labels added: VBUS1, VBUS1_S, VBUS2, VBUS2_S, VBUS3, VBUS3_S
- wire segments 81 -> 116
Other:
- note added: "Power switches"
- note added: "TODO: add 3x USB 2.0 type A connectors (vertical right-angle)"
- note added: "TODO: connect GPIOs to peripherals"
- note added: "TODO: decide what to do with unconnected nets"
- note added: "TODO: decide whether it's better to connect to 3V3 or 5V0"
- note removed: "TODO: add VBUS power controller"

Commit message: Add 3x vertical USB connector
Parts:
- added J? (x3): 73725-0110BLF, antmicro-footprints:USB_A_Female_Vertical_RA_73725-0110BLF, symbol antmicroUSBDVIHDMIConnectors:73725-0110BLF
Connections:
- wire segments 116 -> 141
Other:
- note removed: "TODO: add 3x USB 2.0 type A connectors (vertical right-angle)"
Changed lines of the file:
@@
 Text Notes 2950 2650 0    50   ~ 0
 TODO: connect GPIOs to peripherals
-Text Notes 12875 2150 0    50   ~ 0
-TODO: add 3x USB 2.0 type A connectors (vertical right-angle)
+Wire Wire Line
+	3700 2200 4275 2200
+Text Label 4275 2200 2    50   ~ 0
+RESET_N
+$Comp
+L antmicroUSBDVIHDMIConnectors:73725-0110BLF J?
+U 1 1 60449899
+P 13300 3575
+F 0 "J?" H 13420 4087 60  0000 C CNN
+F 1 "73725-0110BLF" H 13420 3981 60  0000 C CNN
+F 2 "antmicro-footprints:USB_A_Female_Vertical_RA_73725-0110BLF" H 13500 3775 60  0001 L CNN
+F 3 "http://www.amphenol-icc.com/media/wysiwyg/files/drawing/73725.pdf" H 13500 3875 60  0001 L CNN
+F 4 "73725-0110BLF" H 13500 4075 60  0001 L CNN "MPN"
+F 5 "Amphenol ICC (FCI)" H 13500 4675 60  0001 L CNN "Manufacturer"
+	1    13300 3575
+	1    0    0    -1
+$EndComp
+$Comp
+L antmicroUSBDVIHDMIConnectors:73725-0110BLF J?
+U 1 1 6044A36C
+P 13275 4950
+F 0 "J?" H 13395 5462 60  0000 C CNN
+F 1 "73725-0110BLF" H 13400 5350 60  0000 C CNN
+F 2 "antmicro-footprints:USB_A_Female_Vertical_RA_73725-0110BLF" H 13475 5150 60  0001 L CNN
+F 3 "http://www.amphenol-icc.com/media/wysiwyg/files/drawing/73725.pdf" H 13475 5250 60  0001 L CNN
+F 4 "73725-0110BLF" H 13475 5450 60  0001 L CNN "MPN"
+F 5 "Amphenol ICC (FCI)" H 13475 6050 60  0001 L CNN "Manufacturer"
+	1    13275 4950
+	1    0    0    -1
+$EndComp
+$Comp
+L antmicroUSBDVIHDMIConnectors:73725-0110BLF J?
+U 1 1 6044BF40
+P 13300 6300
+F 0 "J?" H 13420 6812 60  0000 C CNN
+F 1 "73725-0110BLF" H 13420 6706 60  0000 C CNN
+F 2 "antmicro-footprints:USB_A_Female_Vertical_RA_73725-0110BLF" H 13500 6500 60  0001 L CNN
+F 3 "http://www.amphenol-icc.com/media/wysiwyg/files/drawing/73725.pdf" H 13500 6600 60  0001 L CNN
+F 4 "73725-0110BLF" H 13500 6800 60  0001 L CNN "MPN"
+F 5 "Amphenol ICC (FCI)" H 13500 7400 60  0001 L CNN "Manufacturer"
+	1    13300 6300
+	1    0    0    -1
+$EndComp
+Wire Wire Line
+	13600 3475 14150 3475
+Wire Wire Line
+	13600 3575 14150 3575
+Text Label 14150 3475 2    50   ~ 0
+USB1_D_N
+Text Label 14150 3575 2    50   ~ 0
+USB1_D_P
+Wire Wire Line
+	13575 4850 14125 4850
+Wire Wire Line
+	13575 4950 14125 4950
+Text Label 14125 4950 2    50   ~ 0
+USB2_D_N
+Text Label 14125 4850 2    50   ~ 0
+USB2_D_P
+Wire Wire Line
+	13600 6200 14150 6200
+Wire Wire Line
+	13600 6300 14150 6300
+Text Label 14150 6200 2    50   ~ 0
+USB3_D_N
+Text Label 14150 6300 2    50   ~ 0
+USB3_D_P
+Wire Wire Line
+	13575 4750 13700 4750
+Wire Wire Line
+	13400 5275 13400 5425
+Wire Wire Line
+	13400 5425 13700 5425
+Wire Wire Line
+	13700 4750 13700 5425
+Wire Wire Line
+	13700 5425 13700 5500
+Connection ~ 13700 5425
+$Comp
+L power:GND #PWR?
+U 1 1 6048FF7A
+P 13700 5500
+F 0 "#PWR?" H 13700 5250 50  0001 C CNN
+F 1 "GND" H 13705 5327 50  0000 C CNN
+F 2 "" H 13700 5500 50  0001 C CNN
+F 3 "" H 13700 5500 50  0001 C CNN
+	1    13700 5500
+	1    0    0    -1
+$EndComp
+Text GLabel 14100 5050 2    50   Input ~ 0
+VCC5V0
+Wire Wire Line
+	13575 5050 14100 5050
+Wire Wire Line
+	13600 3375 13725 3375
+Wire Wire Line
+	13425 3900 13425 4050
+Wire Wire Line
+	13425 4050 13725 4050
+Wire Wire Line
+	13725 3375 13725 4050
+Wire Wire Line
+	13725 4050 13725 4125
+Connection ~ 13725 4050
+$Comp
+L power:GND #PWR?
+U 1 1 604BD8F1
+P 13725 4125
+F 0 "#PWR?" H 13725 3875 50  0001 C CNN
+F 1 "GND" H 13730 3952 50  0000 C CNN
+F 2 "" H 13725 4125 50  0001 C CNN
+F 3 "" H 13725 4125 50  0001 C CNN
+	1    13725 4125
+	1    0    0    -1
+$EndComp
+Text GLabel 14125 3675 2    50   Input ~ 0
+VCC5V0
+Wire Wire Line
+	13600 3675 14125 3675
+Wire Wire Line
+	13600 6100 13725 6100
+Wire Wire Line
+	13425 6625 13425 6775
+Wire Wire Line
+	13425 6775 13725 6775
+Wire Wire Line
+	13725 6100 13725 6775
+Wire Wire Line
+	13725 6775 13725 6850
+Connection ~ 13725 6775
+$Comp
+L power:GND #PWR?
+U 1 1 604C3EB2
+P 13725 6850
+F 0 "#PWR?" H 13725 6600 50  0001 C CNN
+F 1 "GND" H 13730 6677 50  0000 C CNN
+F 2 "" H 13725 6850 50  0001 C CNN
+F 3 "" H 13725 6850 50  0001 C CNN
+	1    13725 6850
+	1    0    0    -1
+$EndComp
+Text GLabel 14125 6400 2    50   Input ~ 0
+VCC5V0
+Wire Wire Line
+	13600 6400 14125 6400
 $EndSCHEMATC

Commit message: Add changes to schematic
-Add pull up resistors on I2C
-Add Voltage devider on VBUS_DET
-Add Hi-Speed upstream port indicator LED
Parts:
- added D?: LG_L29K-G2J1-24-Z, antmicro-footprints:LED_0603, symbol antmicroLEDIndicationDiscrete:LG_L29K-G2J1-24-Z
- added R? (x2): R_100k_0402, antmicro-footprints:0402-res, symbol antmicroResistors0402:R_100k_0402
- added R? (x4): R_10k_0402, antmicro-footprints:0402-res, symbol antmicroResistors0402:R_10k_0402
- added R?: R_47k_0402, antmicro-footprints:0402-res, symbol antmicroResistors0402:R_47k_0402
Connections:
- net labels added: HS_IND, SLOW_~ALERT, ~PWRDN
- wire segments 141 -> 172
- no-connect marks 2 -> 4
Other:
- note added: "High Speed Indicator"
- note added: "TODO:Decide what to do with these pins"
- note added: "USB A connectors"

Commit message: Update schematic
Parts:
- gave numbers to parts that had none: 31

Commit message: Add FTDI and clean up schematic
Parts:
- removed R10, R11: R_10k_0402, antmicro-footprints:0402-res, symbol antmicroResistors0402:R_10k_0402
- added 3V0?, 5V0?: TP_SMD1MM, antartix-arty-controller-footprints:Testpoint_smd_1mm, symbol antartix-arty-controller:TP_SMD1MM
- added C? (x16): C_100n_0402, antartix-arty-controller-footprints:0402-cap, symbol antartix-arty-controller:C_100n_0402
- added C? (x2): C_22p_0402, antartix-arty-controller-footprints:0402-cap, symbol antartix-arty-controller:C_22p_0402
- added D?: TPD2E009, antartix-arty-controller-footprints:SOT-3, symbol antartix-arty-controller:TPD2E009
- added D? (x4): LG_L29K-G2J1-24-Z, antartix-arty-controller-footprints:LED_0603, symbol antartix-arty-controller:LG_L29K-G2J1-24-Z
- added FB?: BLM18PG121SN1D, antartix-arty-controller-footprints:0603-res, symbol antartix-arty-controller:BLM18PG121SN1D
- added IC?: FT2232D, antartix-arty-controller-footprints:LQFP-48_7x7mm, symbol antartix-arty-controller:FT2232D
- added J?: WE_629105150521, antartix-arty-controller-footprints:USB_Micro_B_Female_629105150521, symbol antartix-arty-controller:WE_629105150521
- added R? (x8): R_0R_0402, antartix-arty-controller-footprints:0402-res, symbol antartix-arty-controller:R_0R_0402
- added R?: R_220R_0402, antartix-arty-controller-footprints:0402-res, symbol antartix-arty-controller:R_220R_0402
- added R? (x5): R_470R_0402, antartix-arty-controller-footprints:0402-res, symbol antartix-arty-controller:R_470R_0402
- added R?: R_1k54_0402, antartix-arty-controller-footprints:0402-res, symbol antartix-arty-controller:R_1k54_0402
- added R?: R_4k7_0402, antartix-arty-controller-footprints:0402-res, symbol antartix-arty-controller:R_4k7_0402
- added R?: R_10k_0402, antartix-arty-controller-footprints:0402-res, symbol antartix-arty-controller:R_10k_0402
- added R?: R_0R01_1206, antartix-arty-controller-footprints:1206-res, symbol antartix-arty-controller:R_0R01_1206
- added U?: TPS2051BDBVR, antartix-arty-controller-footprints:SOT-753, symbol antartix-arty-controller:TPS2051BDBVR
- added Y?: MQ-6.000-12-30_30_, antartix-arty-controller-footprints:Crystal_5x7mm, symbol antartix-arty-controller:MQ-6.000-12-30_30_
- C1, C2, C3, C5, C7: footprint antmicro-footprints:0402-cap -> antartix-arty-controller-footprints:0402-cap; symbol antmicroCapacitors0402:C_100n_0402 -> antartix-arty-controller:C_100n_0402
- C4, C6, C8: footprint antmicro-footprints:0402-cap -> antartix-arty-controller-footprints:0402-cap; symbol antmicroCapacitors0402:C_47p_0402 -> antartix-arty-controller:C_47p_0402
- D1: footprint antmicro-footprints:LED_0603 -> antartix-arty-controller-footprints:LED_0603; symbol antmicroLEDIndicationDiscrete:LG_L29K-G2J1-24-Z -> antartix-arty-controller:LG_L29K-G2J1-24-Z
- J1: footprint antmicro-footprints:QTE-020-04-L-D-A -> antartix-arty-controller-footprints:QTE-020-04-L-D-A; symbol antmicroRectangularConnectorsHeadersFemalePins:QTE-020-04-L-D-A -> antartix-arty-controller:QTE-020-04-L-D-A
- J2, J3, J4: footprint antmicro-footprints:USB_A_Female_Vertical_RA_73725-0110BLF -> antartix-arty-controller-footprints:USB_A_Female_Vertical_RA_73725-0110BLF; symbol antmicroUSBDVIHDMIConnectors:73725-0110BLF -> antartix-arty-controller:73725-0110BLF
- R1: footprint antmicro-footprints:0402-res -> antartix-arty-controller-footprints:0402-res; symbol antmicroResistors0402:R_47k_0402 -> antartix-arty-controller:R_47k_0402
- R2, R3: footprint antmicro-footprints:0402-res -> antartix-arty-controller-footprints:0402-res; symbol antmicroResistors0402:R_100k_0402 -> antartix-arty-controller:R_100k_0402
- R4, R5: footprint antmicro-footprints:0402-res -> antartix-arty-controller-footprints:0402-res; symbol antmicroResistors0402:R_10k_0402 -> antartix-arty-controller:R_10k_0402
- R6, R7, R8: footprint antmicro-footprints:1206-res -> antartix-arty-controller-footprints:1206-res; symbol antmicroResistorsmisc:R_0R01_1206 -> antartix-arty-controller:R_0R01_1206
- R9: footprint antmicro-footprints:0402-res -> antartix-arty-controller-footprints:0402-res; symbol antmicroResistors0402:R_22R_0402 -> antartix-arty-controller:R_22R_0402
- U1: footprint antmicro-footprints:SOT95P275X110-6N -> antartix-arty-controller-footprints:SOT95P275X110-6N; symbol antmicroTemperatureSensorsAnalogandDigitalOutput:PCT2075GVX -> antartix-arty-controller:PCT2075GVX
- U2: footprint antmicro-footprints:QFN65P400X400X55-17N -> antartix-arty-controller-footprints:QFN65P400X400X55-17N; symbol antmicroMicrocontrollers:PAC1934T-I_JQ -> antartix-arty-controller:PAC1934T-I_JQ
- U3: footprint antmicro-footprints:QFN50P600X600X100-37N -> antartix-arty-controller-footprints:QFN50P600X600X100-37N; symbol antmicroInterfaceControllers:USB2514B-I_M2 -> antartix-arty-controller:USB2514B-I_M2
- U4, U5, U6: footprint antmicro-footprints:SOT-753 -> antartix-arty-controller-footprints:SOT-753; symbol antmicroPMICPowerDistributionSwitchesLoadDrivers:TPS2051BDBVR -> antartix-arty-controller:TPS2051BDBVR
- Y1: footprint antmicro-footprints:7C-24.000MBB-T -> antartix-arty-controller-footprints:7C-24.000MBB-T; symbol antmicroOscillators:7C-24.000MBB-T -> antartix-arty-controller:7C-24.000MBB-T
Connections:
- net labels added: FTDI_RST, OC_N4, SCL_FTDI, SDA_FTDI, USB4_EN, USB_D_N_CON, USB_D_N_FTDI, USB_D_P_CON, USB_D_P_FTDI, VBUS4, VBUS4_S, WP_FTDI
- wire segments 172 -> 309
- no-connect marks 4 -> 2
Other:
- note added: "FTDI USB->I2C"
- note added: "FTDI power filtering"
- note added: "Micro USB connector"
- note added: "TODO: check if these pull-ups aren't doubled at NODE side"
- note added: "TODO: decide which of these connect to GPIOs"
- note removed: "TODO: connect GPIOs to peripherals"
- note removed: "TODO: decide what to do with unconnected nets"
- moved on the sheet: J1

Commit message: Fix outline
Parts:
- removed J2, J3, J4: 73725-0110BLF, antartix-arty-controller-footprints:USB_A_Female_Vertical_RA_73725-0110BLF, symbol antartix-arty-controller:73725-0110BLF
- added D?: LG_L29K-G2J1-24-Z, antartix-arty-controller-footprints:LED_0603, symbol antartix-arty-controller:LG_L29K-G2J1-24-Z
- added J2, J3, J4: 614004185023, 614004185023, symbol antmicroUSBDVIHDMIConnectors:614004185023
- added R? (x2): R_0R_0805, antmicro-footprints:0805-res, symbol antmicroResistorsmisc:R_0R_0805
- added R?: R_12k_0402, antmicro-footprints:0402-res, symbol antmicroResistors0402:R_12k_0402
- added R?: R_47k_0402, antartix-arty-controller-footprints:0402-res, symbol antartix-arty-controller:R_47k_0402
- gave numbers to parts that had none: 48
Connections:
- net labels added: 3V3_RPI, 3V3_SSD, SUSP_IND
- net labels removed: GPIO06, GPIO12, GPIO13, GPIO16, GPIO19, GPIO20, GPIO21, GPIO26
- wire segments 309 -> 331
Other:
- note added: "LED indicators"
- note removed: "High Speed Indicator"
- note removed: "TODO: add 3V3 source from Node board"
- note removed: "TODO: check if these pull-ups aren't doubled at NODE side"
- note removed: "TODO: decide whether it's better to connect to 3V3 or 5V0"
- note removed: "TODO: decide which of these connect to GPIOs"
- note removed: "TODO:Decide what to do with these pins"
- moved on the sheet: 3V0, 5V0, D1, R1, R4, R5

Commit message: Update current monitoring circuit
Parts:
- gave numbers to parts that had none: 5
Connections:
- wire segments 331 -> 343
Other:
- moved on the sheet: R14, R6, R7, R8
Changed lines of the file:
@@
 Wire Wire Line
 	7925 8850 7575 8850
-Wire Wire Line
-	5975 8950 5850 8950
-Wire Wire Line
-	5975 9050 5550 9050
-Wire Wire Line
-	5550 9050 5550 8950
-Wire Wire Line
-	5975 9250 5850 9250
-Wire Wire Line
-	5975 9350 5550 9350
-Wire Wire Line
-	5550 9350 5550 9250
-Wire Wire Line
-	5550 8950 5450 8950
-Wire Wire Line
-	5550 9250 5450 9250
-Text GLabel 5450 8950 0    50   Input ~ 0
+Text GLabel 5425 8875 0    50   Input ~ 0
 VBUS2_S
-Text GLabel 5450 9250 0    50   Input ~ 0
+Text GLabel 4575 9175 0    50   Input ~ 0
 VBUS3_S
-Wire Wire Line
-	5550 9050 5450 9050
-Wire Wire Line
-	5550 9350 5450 9350
-Text GLabel 5450 9050 0    50   Input ~ 0
+Text GLabel 5425 9175 0    50   Input ~ 0
 VBUS2
-Text GLabel 5450 9350 0    50   Input ~ 0
+Text GLabel 4575 9475 0    50   Input ~ 0
 VBUS3
-Connection ~ 5550 9050
-Connection ~ 5550 9350
 Wire Wire Line
 	7575 9050 8175 9050
@@
 LED indicators
 Text GLabel 12300 1975 2    50   Input ~ 0
-VBUS1_S
+VBUS1
 Text GLabel 13800 2000 2    50   Input ~ 0
-VBUS2_S
+VBUS2
 Text GLabel 15250 2000 2    50   Input ~ 0
-VBUS3_S
+VBUS3
 Text GLabel 4800 1250 1    50   Input ~ 0
 VCC3V3
@@
 L antartix-arty-controller:R_0R01_1206 R8
 U 1 1 6028CD2F
-P 5700 9250
-F 0 "R8" H 5700 9037 60  0000 C CNN
-F 1 "R_0R01_1206" H 5700 9100 60  0001 C CNN
-F 2 "antartix-arty-controller-footprints:1206-res" H 5900 9450 60  0001 L CNN
-F 3 "" H 5700 9250 50  0001 C CNN
-F 4 "PANASONIC" H 5900 9650 60  0001 L CNN "Manufacturer"
-F 5 "ERJMP2KF10MU" H 5900 9550 60  0001 L CNN "MPN"
-F 6 "0R01" H 5700 9135 50  0000 C CNN "Val"
-	1    5700 9250
-	-1   0    0    1
-$EndComp
-Wire Wire Line
-	5975 8650 5850 8650
+P 4725 9325
+F 0 "R8" H 4725 9112 60  0000 C CNN
+F 1 "R_0R01_1206" H 4725 9175 60  0001 C CNN
+F 2 "antartix-arty-controller-footprints:1206-res" H 4925 9525 60  0001 L CNN
+F 3 "" H 4725 9325 50  0001 C CNN
+F 4 "PANASONIC" H 4925 9725 60  0001 L CNN "Manufacturer"
+F 5 "ERJMP2KF10MU" H 4925 9625 60  0001 L CNN "MPN"
+F 6 "0R01" H 4725 9210 50  0000 C CNN "Val"
+	1    4725 9325
+	0    -1   -1   0
+$EndComp
 $Comp
 L antartix-arty-controller:R_0R01_1206 R7
 U 1 1 6028C64E
-P 5700 8950
-F 0 "R7" H 5700 8737 60  0000 C CNN
-F 1 "R_0R01_1206" H 5700 8800 60  0001 C CNN
-F 2 "antartix-arty-controller-footprints:1206-res" H 5900 9150 60  0001 L CNN
-F 3 "" H 5700 8950 50  0001 C CNN
-F 4 "PANASONIC" H 5900 9350 60  0001 L CNN "Manufacturer"
-F 5 "ERJMP2KF10MU" H 5900 9250 60  0001 L CNN "MPN"
-F 6 "0R01" H 5700 8835 50  0000 C CNN "Val"
-	1    5700 8950
-	-1   0    0    1
+P 4725 8725
+F 0 "R7" H 4725 8512 60  0000 C CNN
+F 1 "R_0R01_1206" H 4725 8575 60  0001 C CNN
+F 2 "antartix-arty-controller-footprints:1206-res" H 4925 8925 60  0001 L CNN
+F 3 "" H 4725 8725 50  0001 C CNN
+F 4 "PANASONIC" H 4925 9125 60  0001 L CNN "Manufacturer"
+F 5 "ERJMP2KF10MU" H 4925 9025 60  0001 L CNN "MPN"
+F 6 "0R01" H 4725 8610 50  0000 C CNN "Val"
+	1    4725 8725
+	0    -1   -1   0
 $EndComp
 $Comp
 L antartix-arty-controller:R_0R01_1206 R6
 U 1 1 6028C199
-P 5700 8650
-F 0 "R6" H 5700 8437 60  0000 C CNN
-F 1 "R_0R01_1206" H 5700 8500 60  0001 C CNN
-F 2 "antartix-arty-controller-footprints:1206-res" H 5900 8850 60  0001 L CNN
-F 3 "" H 5700 8650 50  0001 C CNN
-F 4 "PANASONIC" H 5900 9050 60  0001 L CNN "Manufacturer"
-F 5 "ERJMP2KF10MU" H 5900 8950 60  0001 L CNN "MPN"
-F 6 "0R01" H 5700 8535 50  0000 C CNN "Val"
-	1    5700 8650
-	-1   0    0    1
-$EndComp
-Wire Wire Line
-	5975 8750 5550 8750
-Connection ~ 5550 8750
-Wire Wire Line
-	5550 8750 5550 8650
-Wire Wire Line
-	5450 8750 5550 8750
-Text GLabel 5450 8750 0    50   Input ~ 0
+P 5575 9025
+F 0 "R6" H 5575 8812 60  0000 C CNN
+F 1 "R_0R01_1206" H 5575 8875 60  0001 C CNN
+F 2 "antartix-arty-controller-footprints:1206-res" H 5775 9225 60  0001 L CNN
+F 3 "" H 5575 9025 50  0001 C CNN
+F 4 "PANASONIC" H 5775 9425 60  0001 L CNN "Manufacturer"
+F 5 "ERJMP2KF10MU" H 5775 9325 60  0001 L CNN "MPN"
+F 6 "0R01" H 5575 8910 50  0000 C CNN "Val"
+	1    5575 9025
+	0    -1   -1   0
+$EndComp
+Text GLabel 4575 8875 0    50   Input ~ 0
 VBUS1
 Text Notes 12875 1025 0    118  ~ 0
 USB A connectors
-Wire Wire Line
-	5450 8650 5550 8650
-Text GLabel 5450 8650 0    50   Input ~ 0
+Text GLabel 4575 8575 0    50   Input ~ 0
 VBUS1_S
 $Comp
@@
 	12625 3650 12950 3650
 Text GLabel 14550 3650 2    50   Input ~ 0
-VBUS4_S
+VBUS4
 Wire Wire Line
 	13350 3650 14550 3650
@@
 	12225 4450 12225 4550
 Text GLabel 15750 3500 1    50   Input ~ 0
-VBUS4_S
+VBUS4
 Wire Wire Line
 	15800 2400 15800 2300
@@
 $EndComp
 Text GLabel 15800 1875 1    50   Input ~ 0
-VBUS3_S
+VBUS3
 Wire Notes Line
 	11575 2800 16075 2800
@@
 $EndComp
 Text GLabel 12825 1875 1    50   Input ~ 0
-VBUS1_S
+VBUS1
 Wire Wire Line
 	14325 2425 14325 2325
@@
 $EndComp
 Text GLabel 14325 1900 1    50   Input ~ 0
-VBUS2_S
+VBUS2
 Wire Notes Line
 	4025 475  4025 6600
@@
 Wire Wire Line
 	5975 9550 5850 9550
-Wire Wire Line
-	5975 9650 5550 9650
-Wire Wire Line
-	5550 9650 5550 9550
-Wire Wire Line
-	5550 9550 5450 9550
-Text GLabel 5450 9550 0    50   Input ~ 0
+Text GLabel 5425 9475 0    50   Input ~ 0
 VBUS4_S
-Wire Wire Line
-	5550 9650 5450 9650
-Text GLabel 5450 9650 0    50   Input ~ 0
+Text GLabel 5425 9775 0    50   Input ~ 0
 VBUS4
-Connection ~ 5550 9650
 $Comp
 L antartix-arty-controller:R_0R01_1206 R14
 U 1 1 61B3495C
-P 5700 9550
-F 0 "R14" H 5700 9337 60  0000 C CNN
-F 1 "R_0R01_1206" H 5700 9400 60  0001 C CNN
-F 2 "antartix-arty-controller-footprints:1206-res" H 5900 9750 60  0001 L CNN
-F 3 "" H 5700 9550 50  0001 C CNN
-F 4 "PANASONIC" H 5900 9950 60  0001 L CNN "Manufacturer"
-F 5 "ERJMP2KF10MU" H 5900 9850 60  0001 L CNN "MPN"
-F 6 "0R01" H 5700 9435 50  0000 C CNN "Val"
-	1    5700 9550
-	-1   0    0    1
+P 5575 9625
+F 0 "R14" H 5575 9412 60  0000 C CNN
+F 1 "R_0R01_1206" H 5575 9475 60  0001 C CNN
+F 2 "antartix-arty-controller-footprints:1206-res" H 5775 9825 60  0001 L CNN
+F 3 "" H 5575 9625 50  0001 C CNN
+F 4 "PANASONIC" H 5775 10025 60  0001 L CNN "Manufacturer"
+F 5 "ERJMP2KF10MU" H 5775 9925 60  0001 L CNN "MPN"
+F 6 "0R01" H 5575 9510 50  0000 C CNN "Val"
+	1    5575 9625
+	0    -1   -1   0
 $EndComp
 $Comp
@@
 	2525 2025 2525 1925
 $Comp
-L antartix-arty-controller:GND #PWR?
+L antartix-arty-controller:GND #PWR0101
 U 1 1 60563464
 P 2800 1925
-F 0 "#PWR?" H 2800 1675 50  0001 C CNN
+F 0 "#PWR0101" H 2800 1675 50  0001 C CNN
 F 1 "GND" V 2805 1797 50  0000 R CNN
 F 2 "" H 2800 1925 50  0001 C CNN
@@
 3V3_SSD
 $Comp
-L antmicroResistorsmisc:R_0R_0805 R?
+L antmicroResistorsmisc:R_0R_0805 R28
 U 1 1 6082F090
 P 1275 3225
-F 0 "R?" H 1150 3325 60  0000 C CNN
+F 0 "R28" H 1150 3325 60  0000 C CNN
 F 1 "R_0R_0805" H 1275 3075 60  0001 C CNN
 F 2 "antmicro-footprints:0805-res" H 1475 3425 60  0001 L CNN
@@
 $EndComp
 $Comp
-L antmicroResistorsmisc:R_0R_0805 R?
+L antmicroResistorsmisc:R_0R_0805 R29
 U 1 1 6082F5D5
 P 1275 3525
-F 0 "R?" H 1150 3650 60  0000 C CNN
+F 0 "R29" H 1150 3650 60  0000 C CNN
 F 1 "R_0R_0805" H 1275 3375 60  0001 C CNN
 F 2 "antmicro-footprints:0805-res" H 1475 3725 60  0001 L CNN
@@
 	1625 1925 1875 1925
 $Comp
-L antmicroResistors0402:R_12k_0402 R?
+L antmicroResistors0402:R_12k_0402 R31
 U 1 1 60A2CDD5
 P 7975 3725
-F 0 "R?" V 8020 3655 60  0000 R CNN
+F 0 "R31" V 8020 3655 60  0000 R CNN
 F 1 "R_12k_0402" H 7975 3575 60  0001 C CNN
 F 2 "antmicro-footprints:0402-res" H 8175 3925 60  0001 L CNN
@@
 	900  8450 1325 8450
 $Comp
-L antartix-arty-controller:R_47k_0402 R?
+L antartix-arty-controller:R_47k_0402 R30
 U 1 1 60AE7F33
 P 1600 8800
-F 0 "R?" V 1555 8870 60  0000 L CNN
+F 0 "R30" V 1555 8870 60  0000 L CNN
 F 1 "R_47k_0402" H 1600 8650 60  0001 C CNN
 F 2 "antartix-arty-controller-footprints:0402-res" H 1800 9000 60  0001 L CNN
@@
 	1325 8800 1450 8800
 $Comp
-L antartix-arty-controller:LG_L29K-G2J1-24-Z D?
+L antartix-arty-controller:LG_L29K-G2J1-24-Z D7
 U 1 1 60AE7F3C
 P 1550 8450
-F 0 "D?" V 1400 8550 60  0000 L CNN
+F 0 "D7" V 1400 8550 60  0000 L CNN
 F 1 "LG_L29K-G2J1-24-Z" H 275 8300 60  0000 L CNN
 F 2 "antartix-arty-controller-footprints:LED_0603" H 1750 8650 60  0001 L CNN
@@
 Text Label 900  8450 0    50   ~ 0
 SUSP_IND
+Wire Wire Line
+	5850 9550 5850 9475
+Wire Wire Line
+	5850 9475 5575 9475
+Wire Wire Line
+	5975 9650 5850 9650
+Wire Wire Line
+	5850 9650 5850 9775
+Wire Wire Line
+	5850 9775 5575 9775
+Wire Wire Line
+	5000 9250 5000 9175
+Wire Wire Line
+	5000 9175 4725 9175
+Wire Wire Line
+	5000 9350 5000 9475
+Wire Wire Line
+	5000 9475 4725 9475
+Wire Wire Line
+	5000 9250 5975 9250
+Wire Wire Line
+	5000 9350 5975 9350
+Wire Wire Line
+	4725 9175 4575 9175
+Wire Wire Line
+	4725 9475 4575 9475
+Connection ~ 4725 9175
+Connection ~ 4725 9475
+Wire Wire Line
+	5975 8950 5850 8950
+Wire Wire Line
+	5850 8950 5850 8875
+Wire Wire Line
+	5975 9050 5850 9050
+Wire Wire Line
+	5850 9050 5850 9175
+Connection ~ 5575 9775
+Connection ~ 5575 9475
+Wire Wire Line
+	5575 9775 5425 9775
+Wire Wire Line
+	5575 9475 5425 9475
+Wire Wire Line
+	5850 9175 5575 9175
+Wire Wire Line
+	5850 8875 5575 8875
+Wire Wire Line
+	5575 9175 5425 9175
+Wire Wire Line
+	5575 8875 5425 8875
+Connection ~ 5575 9175
+Connection ~ 5575 8875
+Wire Wire Line
+	5000 8650 5000 8575
+Wire Wire Line
+	5000 8575 4725 8575
+Wire Wire Line
+	5000 8750 5000 8875
+Wire Wire Line
+	5000 8875 4725 8875
+Wire Wire Line
+	5000 8650 5975 8650
+Wire Wire Line
+	5000 8750 5975 8750
+Wire Wire Line
+	4725 8575 4575 8575
+Wire Wire Line
+	4725 8875 4575 8875
+Connection ~ 4725 8575
+Connection ~ 4725 8875
 $EndSCHEMATC
