File: antartix-arty-controller.sch (KiCad schematic (older format))
At the start: 82 parts, among them IC1 FT2232D, J1 QTE-020-04-L-D-A, J2 614004185023, J3 614004185023, J4 614004185023, J5 WE_629105150521, U1 PCT2075GVX, U2 PAC1934T-I_JQ, U3 USB2514B-I_M2, U4 TPS2051BDBVR, U5 TPS2051BDBVR, U6 TPS2051BDBVR, U7 TPS2051BDBVR, Y1 7C-24.000MBB-T, Y2 MQ-6.000-12-30_30_

Commit message: Layout update (WIP)
Parts:
- added C27: C_100n_0402, antartix-arty-controller-footprints:0402-cap, symbol antartix-arty-controller:C_100n_0402
Connections:
- net labels added: SNS1_N, SNS1_P, SNS2_N, SNS2_P, SNS3_N, SNS3_P, SNS4_N, SNS4_P, USB_D_CON_N, USB_D_CON_P, USB_D_FTDI_N, USB_D_FTDI_P
- net labels removed: USB_D_N_CON, USB_D_N_FTDI, USB_D_P_CON, USB_D_P_FTDI
- wire segments 343 -> 345
