File: antartix-arty-controller.sch (KiCad schematic (older format))
At the start: 83 parts, among them IC1 FT2232D, J1 QTE-020-04-L-D-A, J2 614004185023, J3 614004185023, J4 614004185023, J5 WE_629105150521, U1 PCT2075GVX, U2 PAC1934T-I_JQ, U3 USB2514B-I_M2, U4 TPS2051BDBVR, U5 TPS2051BDBVR, U6 TPS2051BDBVR, U7 TPS2051BDBVR, Y1 7C-24.000MBB-T, Y2 MQ-6.000-12-30_30_

Commit message: Fix optional micro USB connection
Connections:
- net labels added: RP_USB_N, RP_USB_P
- net labels removed: Arty_USB_N, Arty_USB_P
- wire segments 345 -> 349
Other:
- moved on the sheet: R23, R24
Changed lines of the file:
@@
 $EndComp
 Text GLabel 1650 2325 0    50   Input ~ 0
-Arty_USB_P
+RP_USB_P
 Text GLabel 1650 2425 0    50   Input ~ 0
-Arty_USB_N
+RP_USB_N
 Text GLabel 1500 1925 0    50   Input ~ 0
 VCC5V0
@@
 USB3_D_P
 Text GLabel 7975 1975 2    50   Input ~ 0
-Arty_USB_P
+RP_USB_P
 Text GLabel 7975 2075 2    50   Input ~ 0
-Arty_USB_N
+RP_USB_N
 Wire Wire Line
 	7825 1975 7975 1975
@@
 Text Label 5225 2875 0    50   ~ 0
 USB4_EN
-Wire Wire Line
-	14875 4575 14200 4575
-Wire Wire Line
-	14875 4675 14200 4675
-Text Label 14200 4675 0    50   ~ 0
-USB_D_FTDI_P
-Text Label 14200 4575 0    50   ~ 0
-USB_D_FTDI_N
 $Comp
 L antartix-arty-controller:R_0R_0402 R24
 U 1 1 60AD6937
-P 15025 4675
-F 0 "R24" H 14875 4725 60  0000 C CNN
-F 1 "R_0R_0402" H 15025 4525 60  0001 C CNN
-F 2 "antartix-arty-controller-footprints:0402-res" H 15225 4875 60  0001 L CNN
-F 3 "" H 15025 4675 50  0001 C CNN
-F 4 "PANASONIC" H 15225 5075 60  0001 L CNN "Manufacturer"
-F 5 "ERJ2GE0R00X" H 15225 4975 60  0001 L CNN "MPN"
-F 6 "0R" H 15200 4625 50  0000 C CNN "Val"
-	1    15025 4675
-	1    0    0    -1
+P 1275 2075
+F 0 "R24" H 1075 2025 60  0000 C CNN
+F 1 "R_0R_0402" H 1275 1925 60  0001 C CNN
+F 2 "antartix-arty-controller-footprints:0402-res" H 1475 2275 60  0001 L CNN
+F 3 "" H 1275 2075 50  0001 C CNN
+F 4 "PANASONIC" H 1475 2475 60  0001 L CNN "Manufacturer"
+F 5 "ERJ2GE0R00X" H 1475 2375 60  0001 L CNN "MPN"
+F 6 "0R" H 925 2025 50  0000 C CNN "Val"
+	1    1275 2075
+	-1   0    0    1
 $EndComp
 $Comp
 L antartix-arty-controller:R_0R_0402 R23
 U 1 1 60AD8374
-P 15025 4575
-F 0 "R23" H 14875 4625 60  0000 C CNN
-F 1 "R_0R_0402" H 15025 4425 60  0001 C CNN
-F 2 "antartix-arty-controller-footprints:0402-res" H 15225 4775 60  0001 L CNN
-F 3 "" H 15025 4575 50  0001 C CNN
-F 4 "PANASONIC" H 15225 4975 60  0001 L CNN "Manufacturer"
-F 5 "ERJ2GE0R00X" H 15225 4875 60  0001 L CNN "MPN"
-F 6 "0R" H 15200 4525 50  0000 C CNN "Val"
-	1    15025 4575
-	1    0    0    -1
+P 1275 2175
+F 0 "R23" H 1075 2125 60  0000 C CNN
+F 1 "R_0R_0402" H 1275 2025 60  0001 C CNN
+F 2 "antartix-arty-controller-footprints:0402-res" H 1475 2375 60  0001 L CNN
+F 3 "" H 1275 2175 50  0001 C CNN
+F 4 "PANASONIC" H 1475 2575 60  0001 L CNN "Manufacturer"
+F 5 "ERJ2GE0R00X" H 1475 2475 60  0001 L CNN "MPN"
+F 6 "0R" H 925 2125 50  0000 C CNN "Val"
+	1    1275 2175
+	-1   0    0    1
 $EndComp
 Wire Wire Line
@@
 USB_D_FTDI_N
 Wire Wire Line
-	15175 4575 15925 4575
-Wire Wire Line
-	15175 4675 15925 4675
-Text Label 15925 4675 2    50   ~ 0
+	1125 2175 550  2175
+Wire Wire Line
+	1125 2075 550  2075
+Text Label 575  2075 0    50   ~ 0
 USB_D_CON_P
-Text Label 15925 4575 2    50   ~ 0
+Text Label 575  2175 0    50   ~ 0
 USB_D_CON_N
 $Comp
@@
 $EndComp
 Wire Wire Line
-	1950 2325 1650 2325
-Wire Wire Line
-	1950 2425 1650 2425
+	1950 2325 1800 2325
+Wire Wire Line
+	1950 2425 1725 2425
 Wire Wire Line
 	1950 2225 1875 2225
@@
 	900  3625 900  3525
 Connection ~ 900  3525
+Wire Wire Line
+	1425 2175 1725 2175
+Wire Wire Line
+	1725 2175 1725 2425
+Connection ~ 1725 2425
+Wire Wire Line
+	1725 2425 1650 2425
+Wire Wire Line
+	1800 2325 1800 2075
+Wire Wire Line
+	1800 2075 1425 2075
+Connection ~ 1800 2325
+Wire Wire Line
+	1800 2325 1650 2325
 $EndSCHEMATC

Commit message: Component placement done
Parts:
- added C? (x8): C_100n_0402, antartix-arty-controller-footprints:0402-cap, symbol antartix-arty-controller:C_100n_0402
- added C? (x4): C_22u_0603, antmicro-footprints:0603-cap, symbol antmicroCapacitors0603:C_22u_0603
- added R? (x4): R_4k7_0402, antartix-arty-controller-footprints:0402-res, symbol antartix-arty-controller:R_4k7_0402
Connections:
- wire segments 349 -> 357
Other:
- moved on the sheet: C10, C11, C12, C13, C14, C15, C16, C17, C18, C9

Commit message: Modified layout, routed USB. Now routing current sensing
Parts:
- removed C? (x4): C_100n_0402, antartix-arty-controller-footprints:0402-cap, symbol antartix-arty-controller:C_100n_0402
- added C? (x4): C_100n_0603, antmicro-footprints:0603-cap, symbol antmicroCapacitors0603:C_100n_0603
- added N1: antmicro_logo, antmicro-footprints:antmicro-logo_scaled_15mm, symbol antmicroMechanicalParts:antmicro_logo
- added N2: oshw_logo, antmicro-footprints:oshw-logo, symbol antmicroMechanicalParts:oshw_logo
- added R36, R37: R_220R_0402, antartix-arty-controller-footprints:0402-res, symbol antartix-arty-controller:R_220R_0402
- gave numbers to parts that had none: 12
Connections:
- wire segments 357 -> 382
Other:
- moved on the sheet: C10, C11, C12, C13, C14, C15, C16, C17, C18, C2, C3, C32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

Commit message: Problem with power switches
Parts:
- gave numbers to parts that had none: 4
Changed lines of the file:
@@
 Wire Wire Line
 	4475 3400 5450 3400
-Wire Wire Line
-	5975 9550 5400 9550
 $Comp
 L antartix-arty-controller:R_0R01_1206 R14
@@
 	5400 9475 5125 9475
 Wire Wire Line
-	5975 9650 5400 9650
-Wire Wire Line
 	5400 9650 5400 9775
 Wire Wire Line
@@
 Wire Wire Line
 	4525 9475 4250 9475
-Wire Wire Line
-	4525 9250 5975 9250
-Wire Wire Line
-	4525 9350 5975 9350
 Wire Wire Line
 	4250 9175 4100 9175
@@
 Connection ~ 4250 9475
 Wire Wire Line
-	5975 8950 5400 8950
-Wire Wire Line
 	5400 8950 5400 8875
-Wire Wire Line
-	5975 9050 5400 9050
 Wire Wire Line
 	5400 9050 5400 9175
@@
 	9100 2850 9225 2850
 $Comp
-L antmicroCapacitors0603:C_100n_0603 C?
+L antmicroCapacitors0603:C_100n_0603 C29
 U 1 1 610BE8A4
 P 9225 3050
-F 0 "C?" H 9340 3095 60  0000 L CNN
+F 0 "C29" H 9340 3095 60  0000 L CNN
 F 1 "C_100n_0603" H 9225 2900 60  0001 C CNN
 F 2 "antmicro-footprints:0603-cap" H 9425 3250 60  0001 L CNN
@@
 	9100 1750 9225 1750
 $Comp
-L antartix-arty-controller:GND #PWR?
+L antartix-arty-controller:GND #PWR0122
 U 1 1 6118428C
 P 9225 2175
-F 0 "#PWR?" H 9225 1925 50  0001 C CNN
+F 0 "#PWR0122" H 9225 1925 50  0001 C CNN
 F 1 "GND" H 9230 2002 50  0000 C CNN
 F 2 "" H 9225 2175 50  0001 C CNN
@@
 $EndComp
 $Comp
-L antmicroCapacitors0603:C_100n_0603 C?
+L antmicroCapacitors0603:C_100n_0603 C28
 U 1 1 611846BB
 P 9225 1950
-F 0 "C?" H 9340 1995 60  0000 L CNN
+F 0 "C28" H 9340 1995 60  0000 L CNN
 F 1 "C_100n_0603" H 9225 1800 60  0001 C CNN
 F 2 "antmicro-footprints:0603-cap" H 9425 2150 60  0001 L CNN
@@
 	9225 1750 9400 1750
 $Comp
-L antartix-arty-controller:GND #PWR?
+L antartix-arty-controller:GND #PWR0123
 U 1 1 611C9C34
 P 9225 4525
-F 0 "#PWR?" H 9225 4275 50  0001 C CNN
+F 0 "#PWR0123" H 9225 4275 50  0001 C CNN
 F 1 "GND" H 9230 4352 50  0000 C CNN
 F 2 "" H 9225 4525 50  0001 C CNN
@@
 $EndComp
 $Comp
-L antmicroCapacitors0603:C_100n_0603 C?
+L antmicroCapacitors0603:C_100n_0603 C30
 U 1 1 611CA211
 P 9225 4300
-F 0 "C?" H 9340 4345 60  0000 L CNN
+F 0 "C30" H 9340 4345 60  0000 L CNN
 F 1 "C_100n_0603" H 9225 4150 60  0001 C CNN
 F 2 "antmicro-footprints:0603-cap" H 9425 4500 60  0001 L CNN
@@
 	9225 4100 9425 4100
 $Comp
-L antartix-arty-controller:GND #PWR?
+L antartix-arty-controller:GND #PWR0125
 U 1 1 6121FD95
 P 9225 5800
-F 0 "#PWR?" H 9225 5550 50  0001 C CNN
+F 0 "#PWR0125" H 9225 5550 50  0001 C CNN
 F 1 "GND" H 9230 5627 50  0000 C CNN
 F 2 "" H 9225 5800 50  0001 C CNN
@@
 $EndComp
 $Comp
-L antmicroCapacitors0603:C_100n_0603 C?
+L antmicroCapacitors0603:C_100n_0603 C31
 U 1 1 612201C0
 P 9225 5575
-F 0 "C?" H 9340 5620 60  0000 L CNN
+F 0 "C31" H 9340 5620 60  0000 L CNN
 F 1 "C_100n_0603" H 9225 5425 60  0001 C CNN
 F 2 "antmicro-footprints:0603-cap" H 9425 5775 60  0001 L CNN
@@
 Wire Wire Line
 	9225 5375 9450 5375
+Wire Wire Line
+	5975 9050 5400 9050
+Wire Wire Line
+	5975 8950 5400 8950
+Wire Wire Line
+	4525 9350 5975 9350
+Wire Wire Line
+	4525 9250 5975 9250
+Wire Wire Line
+	5975 9650 5400 9650
+Wire Wire Line
+	5975 9550 5400 9550
 $EndSCHEMATC

Commit message: Replace power switches
Parts:
- removed R32, R33, R34, R35: R_4k7_0402, antartix-arty-controller-footprints:0402-res, symbol antartix-arty-controller:R_4k7_0402
- removed U4, U5, U6: TPS2051BDBVR, antartix-arty-controller-footprints:SOT-753, symbol antartix-arty-controller:TPS2051BDBVR
- added R? (x4): R_4k7_0402, antartix-arty-controller-footprints:0402-res, symbol antartix-arty-controller:R_4k7_0402
- added U4, U5, U6: TPS2024DR, antartix-arty-controller-footprints:SOIC-8_W3.9mm, symbol antartix-arty-controller:TPS2024DR
Connections:
- wire segments 382 -> 440
Other:
- moved on the sheet: C10, C11, C12, C13, C14, C15, C16, C17, C18, C2, C3, C31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

Commit message: Routing control signals
Parts:
- gave numbers to parts that had none: 4
Other:
- moved on the sheet: C29, C30, C31, C32, C33, C35, C36, C37, C39, C7, R14, R6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

Commit message: Board routed
Parts:
- added C40: C_1u_0402, antmicro-footprints:0402-cap, symbol antmicroCapacitors0402:C_1u_0402
- added C41, C42, C43, C44, C45, C46: C_100n_0402, antartix-arty-controller-footprints:0402-cap, symbol antartix-arty-controller:C_100n_0402
- added C47, C48, C49: C_330u_KEMET_D, antmicro-footprints:KEMET_D, symbol antmicroCapacitorspol:C_330u_KEMET_D
- added C50: C_680u_KEMET_D, antmicro-footprints:KEMET_D, symbol antmicroCapacitorspol:C_680u_KEMET_D
- added GND (x2): TP_SMD1MM, antartix-arty-controller-footprints:Testpoint_smd_1mm, symbol antartix-arty-controller:TP_SMD1MM
Connections:
- wire segments 440 -> 464
Other:
- note added: "Hub power filtering"

Commit message: review amendments
Parts:
- removed C25, C33: C_100n_0402, antartix-arty-controller-footprints:0402-cap, symbol antartix-arty-controller:C_100n_0402
- removed C31: C_100n_0603, antmicro-footprints:0603-cap, symbol antmicroCapacitors0603:C_100n_0603
- removed C37: C_22u_0603, antmicro-footprints:0603-cap, symbol antmicroCapacitors0603:C_22u_0603
- removed C47, C48, C49: C_330u_KEMET_D, antmicro-footprints:KEMET_D, symbol antmicroCapacitorspol:C_330u_KEMET_D
- removed C50: C_680u_KEMET_D, antmicro-footprints:KEMET_D, symbol antmicroCapacitorspol:C_680u_KEMET_D
- removed FB1: BLM18PG121SN1D, antartix-arty-controller-footprints:0603-res, symbol antartix-arty-controller:BLM18PG121SN1D
- removed R19: R_0R_0402, antartix-arty-controller-footprints:0402-res, symbol antartix-arty-controller:R_0R_0402
- removed R32: R_4k7_0402, antartix-arty-controller-footprints:0402-res, symbol antartix-arty-controller:R_4k7_0402
- removed U7: TPS2051BDBVR, antartix-arty-controller-footprints:SOT-753, symbol antartix-arty-controller:TPS2051BDBVR
- added C31, C33, C37, C47, C48: C_470u_KEMET_D, antartix-arty-controller-footprints:KEMET_D, symbol antartix-arty-controller:C_470u_KEMET_D
- added C49: C_100n_0402, antartix-arty-controller-footprints:0402-cap, symbol antartix-arty-controller:C_100n_0402
- added FB1: BLM21SP111BH1, antartix-arty-controller-footprints:0805-res, symbol antartix-arty-controller:BLM21SP111BH1
- added J6: 0022232041, antmicro-footprints:PinHeader_1x4_P2.54mm_Drill1.02mm, symbol antartix-arty-controller:0022232041
- added R19: R_220R_0402, antartix-arty-controller-footprints:0402-res, symbol antartix-arty-controller:R_220R_0402
- renumbered GND to GND1, GND to GND2
Connections:
- net labels removed: OC_N4, USB4_EN, VBUS4_S
- wire segments 464 -> 458
- no-connect marks 2 -> 4
Other:
- moved on the sheet: C7, D6, R14, R6, R7, R8, U2
