File: aux-power-supply.sch (KiCad schematic (older format))
At the start: 13 parts

Commit message: Add component placement
Parts:
- J9: renamed from J?; footprint (none) -> Connector_Phoenix_MC:PhoenixContact_MCV_1,5_8-G-3.5_1x08_P3.50mm_Vertical
- gave numbers to parts that had none: 12
Changed lines of the file:
@@
 AR Path="/604C47E1/6175AEC0" Ref="Q?"  Part="1"
 AR Path="/60924187/6175AEC0" Ref="Q?"  Part="1"
-F 0 "Q?" H 2650 2207 50  0000 C CNN
+AR Path="/61753C0A/6175AEC0" Ref="Q1"  Part="1"
+F 0 "Q1" H 2650 2207 50  0000 C CNN
 F 1 "FDC6330L" H 2650 2116 50  0000 C CNN
 F 2 "antmicro-footprints:FDC6330L" H 2700 1750 50  0001 L BNN
@@
 AR Path="/604C47E1/6175AEC8" Ref="Q?"  Part="1"
 AR Path="/60924187/6175AEC8" Ref="Q?"  Part="1"
-F 0 "Q?" H 2725 3307 50  0000 C CNN
+AR Path="/61753C0A/6175AEC8" Ref="Q3"  Part="1"
+F 0 "Q3" H 2725 3307 50  0000 C CNN
 F 1 "FDC6330L" H 2725 3216 50  0000 C CNN
 F 2 "antmicro-footprints:FDC6330L" H 2775 2850 50  0001 L BNN
@@
 AR Path="/604C47E1/6175AED0" Ref="Q?"  Part="1"
 AR Path="/60924187/6175AED0" Ref="Q?"  Part="1"
-F 0 "Q?" H 2700 4507 50  0000 C CNN
+AR Path="/61753C0A/6175AED0" Ref="Q2"  Part="1"
+F 0 "Q2" H 2700 4507 50  0000 C CNN
 F 1 "FDC6330L" H 2700 4416 50  0000 C CNN
 F 2 "antmicro-footprints:FDC6330L" H 2750 4050 50  0001 L BNN
@@
 AR Path="/604C47E1/6175AED6" Ref="J?"  Part="1"
 AR Path="/60924187/6175AED6" Ref="J?"  Part="1"
-F 0 "J?" H 2268 5000 50  0000 C CNN
+AR Path="/61753C0A/6175AED6" Ref="J9"  Part="1"
+F 0 "J9" H 2268 5000 50  0000 C CNN
 F 1 "Screw_Terminal_01x08" H 2268 5091 50  0000 C CNN
-F 2 "" H 2350 5625 50  0001 C CNN
+F 2 "Connector_Phoenix_MC:PhoenixContact_MCV_1,5_8-G-3.5_1x08_P3.50mm_Vertical" H 2350 5625 50  0001 C CNN
 F 3 "~" H 2350 5625 50  0001 C CNN
 	1    2350 5625
@@
 U 1 1 6175AEF3
 P 2575 2225
-F 0 "R?" H 2400 2300 60  0000 C CNN
+AR Path="/60924187/6175AEF3" Ref="R?"  Part="1"
+AR Path="/61753C0A/6175AEF3" Ref="R40"  Part="1"
+F 0 "R40" H 2400 2300 60  0000 C CNN
 F 1 "R_1k_0402" H 2575 2075 60  0001 C CNN
 F 2 "antmicro-footprints:0402-res" H 2775 2425 60  0001 L CNN
@@
 U 1 1 6175AF03
 P 3850 1950
-F 0 "R?" H 3850 2163 60  0000 C CNN
+AR Path="/60924187/6175AF03" Ref="R?"  Part="1"
+AR Path="/61753C0A/6175AF03" Ref="R43"  Part="1"
+F 0 "R43" H 3850 2163 60  0000 C CNN
 F 1 "R_100R_0402" H 3850 1800 60  0001 C CNN
 F 2 "antmicro-footprints:0402-res" H 4050 2150 60  0001 L CNN
@@
 U 1 1 6175AF0F
 P 3525 1650
-F 0 "C?" H 3640 1695 60  0000 L CNN
+AR Path="/60924187/6175AF0F" Ref="C?"  Part="1"
+AR Path="/61753C0A/6175AF0F" Ref="C49"  Part="1"
+F 0 "C49" H 3640 1695 60  0000 L CNN
 F 1 "C_10n_0402" H 3525 1500 60  0001 C CNN
 F 2 "antmicro-footprints:0402-cap" H 3725 1850 60  0001 L CNN
@@
 U 1 1 6175AF26
 P 2650 3325
-F 0 "R?" H 2475 3400 60  0000 C CNN
+AR Path="/60924187/6175AF26" Ref="R?"  Part="1"
+AR Path="/61753C0A/6175AF26" Ref="R42"  Part="1"
+F 0 "R42" H 2475 3400 60  0000 C CNN
 F 1 "R_1k_0402" H 2650 3175 60  0001 C CNN
 F 2 "antmicro-footprints:0402-res" H 2850 3525 60  0001 L CNN
@@
 U 1 1 6175AF36
 P 3925 3050
-F 0 "R?" H 3925 3263 60  0000 C CNN
+AR Path="/60924187/6175AF36" Ref="R?"  Part="1"
+AR Path="/61753C0A/6175AF36" Ref="R45"  Part="1"
+F 0 "R45" H 3925 3263 60  0000 C CNN
 F 1 "R_100R_0402" H 3925 2900 60  0001 C CNN
 F 2 "antmicro-footprints:0402-res" H 4125 3250 60  0001 L CNN
@@
 U 1 1 6175AF42
 P 3600 2750
-F 0 "C?" H 3715 2795 60  0000 L CNN
+AR Path="/60924187/6175AF42" Ref="C?"  Part="1"
+AR Path="/61753C0A/6175AF42" Ref="C51"  Part="1"
+F 0 "C51" H 3715 2795 60  0000 L CNN
 F 1 "C_10n_0402" H 3600 2600 60  0001 C CNN
 F 2 "antmicro-footprints:0402-cap" H 3800 2950 60  0001 L CNN
@@
 U 1 1 6175AF59
 P 2625 4525
-F 0 "R?" H 2450 4600 60  0000 C CNN
+AR Path="/60924187/6175AF59" Ref="R?"  Part="1"
+AR Path="/61753C0A/6175AF59" Ref="R41"  Part="1"
+F 0 "R41" H 2450 4600 60  0000 C CNN
 F 1 "R_1k_0402" H 2625 4375 60  0001 C CNN
 F 2 "antmicro-footprints:0402-res" H 2825 4725 60  0001 L CNN
@@
 U 1 1 6175AF69
 P 3900 4250
-F 0 "R?" H 3900 4463 60  0000 C CNN
+AR Path="/60924187/6175AF69" Ref="R?"  Part="1"
+AR Path="/61753C0A/6175AF69" Ref="R44"  Part="1"
+F 0 "R44" H 3900 4463 60  0000 C CNN
 F 1 "R_100R_0402" H 3900 4100 60  0001 C CNN
 F 2 "antmicro-footprints:0402-res" H 4100 4450 60  0001 L CNN
@@
 U 1 1 6175AF75
 P 3575 3950
-F 0 "C?" H 3690 3995 60  0000 L CNN
+AR Path="/60924187/6175AF75" Ref="C?"  Part="1"
+AR Path="/61753C0A/6175AF75" Ref="C50"  Part="1"
+F 0 "C50" H 3690 3995 60  0000 L CNN
 F 1 "C_10n_0402" H 3575 3800 60  0001 C CNN
 F 2 "antmicro-footprints:0402-cap" H 3775 4150 60  0001 L CNN

Commit message: Add FTDI and LEDs
Other:
- note added: "TODO:Replace with 3-794680-8 + 794617-8 + 1-794610-1"
- note added: "TODO:Replace with MC 1,5/ 8-G-3,5 + MCVW 1,5/8-ST-3,5"
Changed lines of the file:
@@
 Text GLabel 1300 3950 0    50   Input ~ 0
 USB3_EN
+Text Notes 2025 6225 0    50   ~ 0
+TODO:Replace with MC 1,5/ 8-G-3,5  + MCVW 1,5/8-ST-3,5
+Text Notes 2000 6575 0    50   ~ 0
+TODO:Replace with  	3-794680-8 + 794617-8 + 1-794610-1
 $EndSCHEMATC
