File: antartix-usb-adapter.sch (KiCad schematic (older format))
At the start: 121 parts, among them IC1 FT2232D, J1 QTE-020-04-L-D-A, J2 0022232041, J20 8-188275-2, J3 614004185023, J4 WE_629105150521, J5 614004185023, J6 614004185023, U1 PCT2075GVX, U2 PAC1934T-I_JQ, U3 USB2514B-I_M2, U4 TPS2024DR, U5 TPS2024DR, U6 TPS2024DR, Y1 7C-24.000MBB-T, Y2 MQ-6.000-12-30_30_

Commit message: Update naming convention
Parts:
- 3V1, 5V1, GND1, GND2: footprint antartix-arty-controller-footprints:Testpoint_smd_1mm -> scalenode-adapter-footprints:Testpoint_smd_1mm; symbol antartix-arty-controller:TP_SMD1MM -> scalenode-adapter:TP_SMD1MM
- C1, C15, C16, C17, C19, C2, C20, C21, C23, C24, C25, C26, C27, C28, C29, C3, C31, C32, C33, C34, C35, C36, C4, C42, C44, C45, C46, C47, C48, C58, C6, C9: footprint antartix-arty-controller-footprints:0402-cap -> scalenode-adapter-footprints:0402-cap; symbol antartix-arty-controller:C_100n_0402 -> scalenode-adapter:C_100n_0402
- C10, C11, C12: footprint antartix-arty-controller-footprints:0603-cap -> scalenode-adapter-footprints:0603-cap; symbol antartix-arty-controller:C_100n_0603 -> scalenode-adapter:C_100n_0603
- C13: footprint antartix-arty-controller-footprints:0402-cap -> scalenode-adapter-footprints:0402-cap; symbol antartix-arty-controller:C_1u_0402 -> scalenode-adapter:C_1u_0402
- C14, C18, C22, C30, C40: footprint antartix-arty-controller-footprints:KEMET_D -> scalenode-adapter-footprints:KEMET_D; symbol antartix-arty-controller:C_470u_KEMET_D -> scalenode-adapter:C_470u_KEMET_D
- C37, C38, C39: footprint antartix-arty-controller-footprints:0603-cap -> scalenode-adapter-footprints:0603-cap; symbol antartix-arty-controller:C_22u_0603 -> scalenode-adapter:C_22u_0603
- C41, C43: footprint antartix-arty-controller-footprints:0402-cap -> scalenode-adapter-footprints:0402-cap; symbol antartix-arty-controller:C_22p_0402 -> scalenode-adapter:C_22p_0402
- C5, C7, C8: footprint antartix-arty-controller-footprints:0402-cap -> scalenode-adapter-footprints:0402-cap; symbol antartix-arty-controller:C_47p_0402 -> scalenode-adapter:C_47p_0402
- D1, D2, D3, D4, D5, D6: footprint antartix-arty-controller-footprints:LED_0603 -> scalenode-adapter-footprints:LED_0603; symbol antartix-arty-controller:LG_L29K-G2J1-24-Z -> scalenode-adapter:LG_L29K-G2J1-24-Z
- D7: footprint antartix-arty-controller-footprints:SOT-3 -> scalenode-adapter-footprints:SOT-3; symbol antartix-arty-controller:TPD2E009 -> scalenode-adapter:TPD2E009
- FB1: footprint antartix-arty-controller-footprints:0805-res -> scalenode-adapter-footprints:0805-res; symbol antartix-arty-controller:BLM21SP111BH1 -> scalenode-adapter:BLM21SP111BH1
- IC1: footprint antartix-arty-controller-footprints:LQFP-48_7x7mm -> scalenode-adapter-footprints:LQFP-48_7x7mm; symbol antartix-arty-controller:FT2232D -> scalenode-adapter:FT2232D
- J1: footprint antartix-arty-controller-footprints:QTE-020-04-L-D-A -> scalenode-adapter-footprints:QTE-020-04-L-D-A; symbol antartix-arty-controller:QTE-020-04-L-D-A -> scalenode-adapter:QTE-020-04-L-D-A
- J2: footprint antartix-arty-controller-footprints:PinHeader_1x4_P2.54mm_Drill1.02mm -> scalenode-adapter-footprints:PinHeader_1x4_P2.54mm_Drill1.02mm; symbol antartix-arty-controller:0022232041 -> scalenode-adapter:0022232041
- J20: footprint antartix-arty-controller-footprints:8-188275-2 -> scalenode-adapter-footprints:8-188275-2; symbol antartix-arty-controller:8-188275-2 -> scalenode-adapter:8-188275-2
- J3, J5, J6: symbol antartix-arty-controller:614004185023 -> scalenode-adapter:614004185023
- J4: footprint antartix-arty-controller-footprints:USB_Micro_B_Female_629105150521 -> scalenode-adapter-footprints:USB_Micro_B_Female_629105150521; symbol antartix-arty-controller:WE_629105150521 -> scalenode-adapter:WE_629105150521
- N1: footprint antartix-arty-controller-footprints:antmicro-logo_scaled_15mm -> scalenode-adapter-footprints:antmicro-logo_scaled_15mm; symbol antartix-arty-controller:antmicro_logo -> scalenode-adapter:antmicro_logo
- N2: footprint antartix-arty-controller-footprints:oshw-logo -> scalenode-adapter-footprints:oshw-logo; symbol antartix-arty-controller:oshw_logo -> scalenode-adapter:oshw_logo
- R1, R2, R31, R32, R33, R35, R36, R52, R53: footprint antartix-arty-controller-footprints:0402-res -> scalenode-adapter-footprints:0402-res; symbol antartix-arty-controller:R_0R_0402 -> scalenode-adapter:R_0R_0402
- R10, R50, R51, R9: footprint antartix-arty-controller-footprints:0402-res -> scalenode-adapter-footprints:0402-res; symbol antartix-arty-controller:R_47k_0402 -> scalenode-adapter:R_47k_0402
- R11, R12, R30, R34: footprint antartix-arty-controller-footprints:0402-res -> scalenode-adapter-footprints:0402-res; symbol antartix-arty-controller:R_220R_0402 -> scalenode-adapter:R_220R_0402
- R13, R14, R27: footprint antartix-arty-controller-footprints:0402-res -> scalenode-adapter-footprints:0402-res; symbol antartix-arty-controller:R_10k_0402 -> scalenode-adapter:R_10k_0402
- R15, R16, R21, R22: footprint antartix-arty-controller-footprints:1206-res -> scalenode-adapter-footprints:1206-res; symbol antartix-arty-controller:R_0R01_1206 -> scalenode-adapter:R_0R01_1206
- R17, R18: footprint antartix-arty-controller-footprints:0402-res -> scalenode-adapter-footprints:0402-res; symbol antartix-arty-controller:R_100k_0402 -> scalenode-adapter:R_100k_0402
- R19, R20, R23, R26: footprint antartix-arty-controller-footprints:0402-res -> scalenode-adapter-footprints:0402-res; symbol antartix-arty-controller:R_4k7_0402 -> scalenode-adapter:R_4k7_0402
- R24, R56, R57: footprint antartix-arty-controller-footprints:0402-res -> scalenode-adapter-footprints:0402-res; symbol antartix-arty-controller:R_22R_0402 -> scalenode-adapter:R_22R_0402
- R25: footprint antartix-arty-controller-footprints:0402-res -> scalenode-adapter-footprints:0402-res; symbol antartix-arty-controller:R_12k_0402 -> scalenode-adapter:R_12k_0402
- R28, R5, R6, R7, R8: footprint antartix-arty-controller-footprints:0402-res -> scalenode-adapter-footprints:0402-res; symbol antartix-arty-controller:R_470R_0402 -> scalenode-adapter:R_470R_0402
- R29: footprint antartix-arty-controller-footprints:0402-res -> scalenode-adapter-footprints:0402-res; symbol antartix-arty-controller:R_1k54_0402 -> scalenode-adapter:R_1k54_0402
- R3, R4: footprint antartix-arty-controller-footprints:0805-res -> scalenode-adapter-footprints:0805-res; symbol antartix-arty-controller:R_0R_0805 -> scalenode-adapter:R_0R_0805
- U1: footprint antartix-arty-controller-footprints:SOT95P275X110-6N -> scalenode-adapter-footprints:SOT95P275X110-6N; symbol antartix-arty-controller:PCT2075GVX -> scalenode-adapter:PCT2075GVX
- U2: footprint antartix-arty-controller-footprints:QFN65P400X400X55-17N -> scalenode-adapter-footprints:QFN65P400X400X55-17N; symbol antartix-arty-controller:PAC1934T-I_JQ -> scalenode-adapter:PAC1934T-I_JQ
- U3: footprint antartix-arty-controller-footprints:QFN50P600X600X100-37N -> scalenode-adapter-footprints:QFN50P600X600X100-37N; symbol antartix-arty-controller:USB2514B-I_M2 -> scalenode-adapter:USB2514B-I_M2
- U4, U5, U6: footprint antartix-arty-controller-footprints:SOIC-8_W3.9mm -> scalenode-adapter-footprints:SOIC-8_W3.9mm; symbol antartix-arty-controller:TPS2024DR -> scalenode-adapter:TPS2024DR
- Y1: footprint antartix-arty-controller-footprints:7C-24.000MBB-T -> scalenode-adapter-footprints:7C-24.000MBB-T; symbol antartix-arty-controller:7C-24.000MBB-T -> scalenode-adapter:7C-24.000MBB-T
- Y2: footprint antartix-arty-controller-footprints:Crystal_5x7mm -> scalenode-adapter-footprints:Crystal_5x7mm; symbol antartix-arty-controller:MQ-6.000-12-30_30_ -> scalenode-adapter:MQ-6.000-12-30_30_
