File: hdmi-adapter.sch (KiCad schematic (older format))
At the start: 46 parts, among them IC2 TPD8S009DSMR, J10 3-794680-8, J11 1-794610-1, J12 1-794610-1, J13 1-794610-1, J14 1-794610-1, J15 794617-8, J16 1-794610-1, J17 1-794610-1, J18 1-794610-1, J19 1-794610-1, J7 QTE-020-04-L-D-A, J8 WE_629105150521, J9 WE_685119136923, Q1 FDC6330L, Q2 FDC6330L, Q3 FDC6330L, U7 FT230XS-R

Commit message: Update naming convention
Parts:
- renumbered C55 to C?, C56 to C?, C57 to C?, J9 to J?, J10 to J?, J16 to J?, J17 to J?, J18 to J?, J19 to J?, J11 to J?, J12 to J?, J13 to J?, J14 to J?, J15 to J?, R54 to R?, R40 to R?, R41 to R?, R55 to R?, R42 to R?, R43 to R?, R44 to R?, R45 to R?, R46 to R?, U7 to U?
