File: usb-adapter.sch (KiCad schematic (older format))
At the start: 121 parts, among them IC1 FT2232D, J1 QTE-020-04-L-D-A, J2 0022232041, J20 8-188275-2, J3 614004185023, J4 WE_629105150521, J5 614004185023, J6 614004185023, U1 PCT2075GVX, U2 PAC1934T-I_JQ, U3 USB2514B-I_M2, U4 TPS2024DR, U5 TPS2024DR, U6 TPS2024DR, Y1 7C-24.000MBB-T, Y2 MQ-6.000-12-30_30_

Commit message: Update naming convention
Parts:
- renumbered J20 to J?, R53 to R?, R52 to R?
